File: Hardware/LibreCAL/LibreCAL.kicad_pcb (KiCad board)
At the start: 4 copper layers, 55 x 73.5 mm, 132 parts, among them J1 901-10510-2, J2 901-10510-2, J3 901-10510-2, J4 901-10510-2, J5 USB_C_Receptacle_USB2.0, J6 TC2030-ARM, Q1 IRLML2060, SW1 TL3301NF160QG, SW2 TL3301CF160QG, SW3 TL3301CF160QG, U1 PE426462, U2 PE426462, U3 PE426462, U4 PE426462, U5 W25Q16JVSNIQ, U6 IP4234CZ6, U7 RP2040, U8 W25Q16JVSNIQ, U9 MIC5528-3.3YMT-TR, Y1 ECS-120-8-36-CKM-TR3

Commit message: LibreCAL Hardware Rev A+ 2023-02-01
Parts:
- R1, R2, R3, R4: value CH0402-50RGFTA -> CH0402-50RGFPT
Routing:
- net +5V: track 81.4 -> 79.9 mm
Other:
- board text added: "JLCPCB 4Layer JLC04161H-7628 Stackup 1.6mm (FR4) Er 4.6 Prepreg Thickness 0.2104mm (0.2mm) CPWG Z=50 Ohms Track width 0.34mm, Conductor Gap 0.2mm Loss about 0.3dB/cm @6GHz Net Name Pad Count Via Count Via Length Track Length Net Length Net loss dB /PortSwitch/U3_RFC_J1 2 0 0.0000 mm 17.5375 mm 17.5375 mm 0.5 /PortSwitch/U1_RFC_J2 2 0 0.0000 mm 17.5375 mm 17.5375 mm 0.5 /PortSwitch/U4_RFC_J3 2 0 0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"
- board text removed: "JLCPCB 4Layer JLC7628 1.6mm Z50Ohms Track width 0.295mm"
