File: Hardware/LibreCAL/PortSwitch.kicad_sch (KiCad schematic)
At the start: 47 parts, among them J1 901-10510-2, J2 901-10510-2, J3 901-10510-2, J4 901-10510-2, U1 PE426462, U2 PE426462, U3 PE426462, U4 PE426462

Commit message: LibreCAL Hardware Rev A+ 2023-02-01
Parts:
- R1, R2, R3, R4: value CH0402-50RGFTA -> CH0402-50RGFPT
Changed lines of the file:
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@@
   (title_block
     (title "LibreCAL")
-    (date "2023-01-07")
+    (date "2023-02-01")
     (rev "A+")
   )
@@
       (effects (font (size 1.27 1.27)) (justify left))
     )
-    (property "Value" "CH0402-50RGFTA" (id 1) (at 166.37 73.6599 0)
+    (property "Value" "CH0402-50RGFPT" (id 1) (at 166.37 73.6599 0)
       (effects (font (size 1.27 1.27)) (justify left))
     )
@@
       (effects (font (size 1.27 1.27)) (justify left))
     )
-    (property "Value" "CH0402-50RGFTA" (id 1) (at 166.37 139.6999 0)
+    (property "Value" "CH0402-50RGFPT" (id 1) (at 166.37 139.6999 0)
       (effects (font (size 1.27 1.27)) (justify left))
     )
@@
       (effects (font (size 1.27 1.27)) (justify left))
     )
-    (property "Value" "CH0402-50RGFTA" (id 1) (at 128.27 139.6999 0)
+    (property "Value" "CH0402-50RGFPT" (id 1) (at 128.27 139.6999 0)
       (effects (font (size 1.27 1.27)) (justify left))
     )
@@
       (effects (font (size 1.27 1.27)) (justify left))
     )
-    (property "Value" "CH0402-50RGFTA" (id 1) (at 128.27 73.6599 0)
-      (effects (font (size 1.27 1.27)) (justify left))
-    )
+    (property "Value" "CH0402-50RGFPT" (id 1) (at 128.27 73.6599 0)
+      (effects (font (size 1.27 1.27)) (justify left))
+    )
